Commit message: create my branch

File: kortex_description/arms/gen3/7dof/urdf/GEN3_URDF_V12.urdf (robot description, URDF)
Before this commit: robot GEN3_URDF_V12, 9 links, 8 joints
Links:
- link base_link: geometry collision mesh filename=package://kortex_description/arms/gen3/meshes/barse_link.STL; visual mesh filename=package://kortex_description/arms/gen3/meshes/base_link.STL
