Commit message: absolute path for non ros sys

File: kortex_description/arms/gen3/7dof/urdf/GEN3_URDF_V12_absPath_pushit.urdf (robot description, URDF)
Before this commit: robot GEN3_URDF_V12, 10 links, 9 joints
Links:
- link Bracelet_Link: geometry collision mesh filename=/home/y/Documents/WYY_META/effectit/ros_kortex/kortex_descr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; visual mesh filename=/home/y/Documents/WYY_META/effectit/ros_kortex/kortex_descr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
- link ForeArm_Link: geometry collision mesh filename=/home/y/Documents/WYY_META/effectit/ros_kortex/kortex_descr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; visual mesh filename=/home/y/Documents/WYY_META/effectit/ros_kortex/kortex_descr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
- link HalfArm1_Link: geometry collision mesh filename=/home/y/Documents/WYY_META/effectit/ros_kortex/kortex_descr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; visual mesh filename=/home/y/Documents/WYY_META/effectit/ros_kortex/kortex_descr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
- link HalfArm2_Link: geometry collision mesh filename=/home/y/Documents/WYY_META/effectit/ros_kortex/kortex_descr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; visual mesh filename=/home/y/Documents/WYY_META/effectit/ros_kortex/kortex_descr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
- link Shoulder_Link: geometry collision mesh filename=/home/y/Documents/WYY_META/effectit/ros_kortex/kortex_descr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; visual mesh filename=/home/y/Documents/WYY_META/effectit/ros_kortex/kortex_descr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
- link SphericalWrist1_Link: geometry collision mesh filename=/home/y/Documents/WYY_META/effectit/ros_kortex/kortex_descr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; visual mesh filename=/home/y/Documents/WYY_META/effectit/ros_kortex/kortex_descr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
- link SphericalWrist2_Link: geometry collision mesh filename=/home/y/Documents/WYY_META/effectit/ros_kortex/kortex_descr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; visual mesh filename=/home/y/Documents/WYY_META/effectit/ros_kortex/kortex_descr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
- link base_link: geometry collision mesh filename=/home/y/Documents/WYY_META/effectit/ros_kortex/kortex_descr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; visual mesh filename=/home/y/Documents/WYY_META/effectit/ros_kortex/kortex_descr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
Joints:
- joint Actuator1: limit effort=39 velocity=0.8727 -> lower=-6.28 upper=6.28 effort=39 velocity=0.8727; type continuous -> revolute
- joint Actuator3: limit effort=39 velocity=0.8727 -> lower=-6.28 upper=6.28 effort=39 velocity=0.8727; type continuous -> revolute
- joint Actuator5: limit effort=9 velocity=0.8727 -> lower=-6.28 upper=6.28 effort=9 velocity=0.8727; type continuous -> revolute
- joint Actuator7: limit effort=9 velocity=0.8727 -> lower=-6.28 upper=6.28 effort=9 velocity=0.8727; type continuous -> revolute
